File: Electrical Desgin/KiCad/Class D Amplifier/Class D Amplifier.kicad_pcb (KiCad board)
At the start: 2 copper layers, 77.5 x 31.8 mm, 27 parts, among them J1 AudioJack3, J2 speakON_NL2MDXX-V, J3 Barrel_Jack, U1 TPA3136D2PWPR

Commit message: pushing PCB changes
Parts:
- removed J1: AudioJack3, Connector_Audio:Jack_3.5mm_CUI_SJ1-3525N_Horizontal
Other:
- board text added: "SUMMED AUDIO IN"
- board text removed: "AUDIO IN"
Changed lines of the file:
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@@
-    )
-  )
-  (footprint "Connector_Audio:Jack_3.5mm_CUI_SJ1-3525N_Horizontal" (layer "F.Cu")
-    (at 116.84 73.66 -90)
-    (descr "TRS 3.5mm, horizontal, through-hole, https://www.cuidevices.com/product/resource/pdf/sj1-352xn.pdf")
-    (tags "TRS audio jack stereo horizontal")
-    (property "Sheetfile" "Class D Amplifier.kicad_sch")
-    (property "Sheetname" "")
-    (property "ki_description" "Audio Jack, 3 Poles (Stereo / TRS)")
-    (property "ki_keywords" "audio jack receptacle stereo headphones phones TRS connector")
-    (attr through_hole exclude_from_pos_files)
-    (fp_text reference "J1" (at 0 -8.8 90) (layer "F.SilkS")
-        (effects (font (size 1 1) (thickness 0.15)))
-    )
-    (fp_text value "AudioJack3" (at 0 -10 90) (layer "F.Fab")
-        (effects (font (size 1 1) (thickness 0.15)))
-    )
-    (fp_text user "PCB edge" (at 0 3.65 -90 unlocked) (layer "Dwgs.User")
-        (effects (font (size 1 1) (thickness 0.15)))
-    )
-    (fp_text user "${REFERENCE}" (at 0 -1.5 90) (layer "F.Fab")
-        (effects (font (size 1 1) (thickness 0.15)))
-    )
-    (fp_line (start -6 -7.7) (end 6 -7.7)
-      (stroke (width 0.12) (type solid)) (layer "F.SilkS"))
-    (fp_line (start -6 3.3) (end -6 -7.7)
-      (stroke (width 0.12) (type solid)) (layer "F.SilkS"))
-    (fp_line (start -4.5 3.3) (end -6 3.3)
-      (stroke (width 0.12) (type solid)) (layer "F.SilkS"))
-    (fp_line (start -4.5 4.5) (end -4.5 3.3)
-      (stroke (width 0.12) (type solid)) (layer "F.SilkS"))
-    (fp_line (start -3 4.5) (end -4.5 4.5)
-      (stroke (width 0.12) (type solid)) (layer "F.SilkS"))
-    (fp_line (start -3 6.3) (end -3 4.5)
-      (stroke (width 0.12) (type solid)) (layer "F.SilkS"))
-    (fp_line (start -2 3.3) (end -2 6.3)
-      (stroke (width 0.12) (type solid)) (layer "F.SilkS"))
-    (fp_line (start 2 3.3) (end -2 3.3)
-      (stroke (width 0.12) (type solid)) (layer "F.SilkS"))
-    (fp_line (start 2 6.3) (end 2 3.3)
-      (stroke (width 0.12) (type solid)) (layer "F.SilkS"))
-    (fp_line (start 3 4.5) (end 3 6.3)
-      (stroke (width 0.12) (type solid)) (layer "F.SilkS"))
-    (fp_line (start 3 6.3) (end -3 6.3)
-      (stroke (width 0.12) (type solid)) (layer "F.SilkS"))
-    (fp_line (start 4.5 3.3) (end 4.5 4.5)
-      (stroke (width 0.12) (type solid)) (layer "F.SilkS"))
-    (fp_line (start 4.5 4.5) (end 3 4.5)
-      (stroke (width 0.12) (type solid)) (layer "F.SilkS"))
-    (fp_line (start 6 -7.7) (end 6 3.3)
-      (stroke (width 0.12) (type solid)) (layer "F.SilkS"))
-    (fp_line (start 6 3.3) (end 4.5 3.3)
-      (stroke (width 0.12) (type solid)) (layer "F.SilkS"))
-    (fp_line (start -2.2 3.5) (end -2.2 4.5)
-      (stroke (width 0.12) (type solid)) (layer "Edge.Cuts"))
-    (fp_line (start -2.2 4.5) (end -6.5 4.5)
-      (stroke (width 0.12) (type solid)) (layer "Edge.Cuts"))
-    (fp_line (start 1.8 3.1) (end -1.8 3.1)
-      (stroke (width 0.12) (type solid)) (layer "Edge.Cuts"))
-    (fp_line (start 2.2 3.5) (end 2.2 4.5)
-      (stroke (width 0.12) (type solid)) (layer "Edge.Cuts"))
-    (fp_line (start 2.2 4.5) (end 6.5 4.5)
-      (stroke (width 0.12) (type solid)) (layer "Edge.Cuts"))
-    (fp_arc (start -2.2 3.5) (mid -2.082842 3.217158) (end -1.8 3.1)
-      (stroke (width 0.12) (type solid)) (layer "Edge.Cuts"))
-    (fp_arc (start 1.8 3.1) (mid 2.082843 3.217157) (end 2.2 3.5)
-      (stroke (width 0.12) (type solid)) (layer "Edge.Cuts"))
-    (fp_line (start -6.25 -7.95) (end -6.25 4.75)
-      (stroke (width 0.05) (type solid)) (layer "F.CrtYd"))
-    (fp_line (start -6.25 4.75) (end -3.25 4.75)
-      (stroke (width 0.05) (type solid)) (layer "F.CrtYd"))
-    (fp_line (start -3.25 4.75) (end -3.25 6.55)
-      (stroke (width 0.05) (type solid)) (layer "F.CrtYd"))
-    (fp_line (start -3.25 6.55) (end 3.25 6.55)
-      (stroke (width 0.05) (type solid)) (layer "F.CrtYd"))
-    (fp_line (start 3.25 4.75) (end 6.25 4.75)
-      (stroke (width 0.05) (type solid)) (layer "F.CrtYd"))
-    (fp_line (start 3.25 6.55) (end 3.25 4.75)
-      (stroke (width 0.05) (type solid)) (layer "F.CrtYd"))
-    (fp_line (start 6.25 -7.95) (end -6.25 -7.95)
-      (stroke (width 0.05) (type solid)) (layer "F.CrtYd"))
-    (fp_line (start 6.25 4.5) (end 6.25 -7.95)
-      (stroke (width 0.05) (type solid)) (layer "F.CrtYd"))
-    (fp_line (start 6.25 4.75) (end 6.25 4.5)
-      (stroke (width 0.05) (type solid)) (layer "F.CrtYd"))
-    (fp_line (start -6 -7.7) (end 6 -7.7)
-      (stroke (width 0.1) (type solid)) (layer "F.Fab"))
-    (fp_line (start -6 3.3) (end -6 -7.7)
-      (stroke (width 0.1) (type solid)) (layer "F.Fab"))
-    (fp_line (start -4.5 3.3) (end -6 3.3)
-      (stroke (width 0.1) (type solid)) (layer "F.Fab"))
-    (fp_line (start -4.5 4.5) (end -4.5 3.3)
-      (stroke (width 0.1) (type solid)) (layer "F.Fab"))
-    (fp_line (start -4.5 4.5) (end -3 4.5)
-      (stroke (width 0.1) (type solid)) (layer "F.Fab"))
-    (fp_line (start -3 4.5) (end -3 6.3)
-      (stroke (width 0.1) (type solid)) (layer "F.Fab"))
-    (fp_line (start -3 6.3) (end 3 6.3)
-      (stroke (width 0.1) (type solid)) (layer "F.Fab"))
-    (fp_line (start 3 4.5) (end 3 6.3)
-      (stroke (width 0.1) (type solid)) (layer "F.Fab"))
-    (fp_line (start 4.5 3.3) (end 6 3.3)
-      (stroke (width 0.1) (type solid)) (layer "F.Fab"))
-    (fp_line (start 4.5 4.5) (end 3 4.5)
-      (stroke (width 0.1) (type solid)) (layer "F.Fab"))
-    (fp_line (start 4.5 4.5) (end 4.5 3.3)
-      (stroke (width 0.1) (type solid)) (layer "F.Fab"))
-    (fp_line (start 6 3.3) (end 6 -7.7)
-      (stroke (width 0.1) (type solid)) (layer "F.Fab"))
-    (pad "" np_thru_hole circle (at -5 0 270) (size 1.2 1.2) (drill 1.2) (layers "*.Cu"))
-    (pad "" np_thru_hole circle (at -5 2.5 270) (size 1.2 1.2) (drill 1.2) (layers "*.Cu"))
-    (pad "" np_thru_hole circle (at 0 -5 270) (size 1.2 1.2) (drill 1.2) (layers "*.Cu"))
-    (pad "" np_thru_hole circle (at 5 0 270) (size 1.2 1.2) (drill 1.2) (layers "*.Cu"))
-    (pad "" np_thru_hole circle (at 5 2.5 270) (size 1.2 1.2) (drill 1.2) (layers "*.Cu"))
-    (pad "R" thru_hole oval (at -5 -5 270) (size 1.2 2.2) (drill oval 0.4 1.4) (layers "*.Cu" "*.Mask")
-      (net 9 "Net-(J1-PadR)") (pintype "passive"))
-    (pad "RN" thru_hole oval (at -2.5 -5 270) (size 1.2 2.2) (drill oval 0.4 1.4) (layers "*.Cu" "*.Mask"))
-    (pad "S" thru_hole oval (at 0 0 270) (size 2.2 1.2) (drill oval 1.4 0.4) (layers "*.Cu" "*.Mask")
-      (net 1 "GND") (pintype "passive"))
-    (pad "T" thru_hole oval (at 5 -5 90) (size 1.2 2.2) (drill oval 0.4 1.4) (layers "*.Cu" "*.Mask")
-      (net 10 "Net-(J1-PadT)") (pintype "passive"))
-    (pad "TN" thru_hole oval (at 2.5 -5 90) (size 1.2 2.2) (drill oval 0.4 1.4) (layers "*.Cu" "*.Mask"))
-    (model "${KICAD6_3DMODEL_DIR}/Connector_Audio.3dshapes/Jack_3.5mm_CUI_SJ1-3525N_Horizontal.wrl"
-      (offset (xyz 0 0 0))
-      (scale (xyz 1 1 1))
-      (rotate (xyz 0 0 0))
     )
   )
@@
   (gr_arc (start 111.76 95.25) (mid 113.556051 95.993949) (end 114.3 97.79)
     (stroke (width 0.1) (type default)) (layer "Edge.Cuts"))
-  (gr_text "AUDIO IN" (at 128.27 73.66 90) (layer "F.SilkS" knockout)
+  (gr_text "SUMMED\nAUDIO IN" (at 129.54 73.66 90) (layer "F.SilkS" knockout)
     (effects (font (size 1 1) (thickness 0.2) bold) (justify bottom))
   )

Commit message: Layout improvements for amp
Parts:
- added J1: AudioJack3, Connector_Audio:Jack_3.5mm_CUI_SJ-3523-SMT_Horizontal, F.Cu at (117.2, 74.8)
- L1, L2: footprint Capacitor_SMD:C_0402_1005Metric_Pad0.74x0.62mm_HandSolder -> Inductor_SMD:L_Taiyo-Yuden_MD-3030
- moved C8 21.0 mm to (131.0, 80.2), turned to 90 degrees
- moved C10 13.8 mm to (139.4, 85.0), turned to 90 degrees
- moved C13 11.7 mm to (153.4, 79.0), turned to 90 degrees
- moved C14 10.5 mm to (153.4, 83.5), turned to -90 degrees
- moved REF** 8.83 mm to (146.0, 89.6)
- moved R3 5.05 mm to (136.6, 90.0)
- moved L1 5.05 mm to (150.3, 79.8)
- moved C11 3.94 mm to (149.6, 77.4)
- moved C12 3.91 mm to (149.6, 86.0), turned to 180 degrees
- moved R4 3.61 mm to (139.4, 90.0), turned to 180 degrees
- moved L2 3.33 mm to (150.3, 83.6)
- moved R5 2.04 mm to (128.8, 79.0)
- moved R2 1.95 mm to (142.0, 87.0), turned to 180 degrees
- moved C9 1.64 mm to (136.8, 86.8)
- moved C5 1.18 mm to (136.4, 72.2)
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