File: Electrical Desgin/KiCad/Class D Amplifier/Class D Amplifier.kicad_sch (KiCad schematic)
At the start: 25 parts, among them J1 AudioJack3, J2 SpeakON_NL2MDXX-V, U1 TPA3136D2PWPR

Commit message: Create PCB files
Parts:
- added J3: Barrel_Jack, Connector_BarrelJack:BarrelJack_CUI_PJ-063AH_Horizontal, symbol Connector:Barrel_Jack
- C1, C13, C14, C2, C3, C4, C5, C9: footprint (none) -> Capacitor_SMD:C_0805_2012Metric_Pad1.18x1.45mm_HandSolder
- C10, C11, C12, C6, C7, C8, L1, L2: footprint (none) -> Capacitor_SMD:C_0402_1005Metric_Pad0.74x0.62mm_HandSolder
- J1: footprint (none) -> Connector_Audio:Jack_3.5mm_CUI_SJ1-3525N_Horizontal
- J2: value SpeakON_NL2MDXX-V -> speakON_NL2MDXX-V; footprint (none) -> Connector_Audio:Jack_speakON_Neutrik_NL2MDXX-H-3_Horizontal
- R1, R2, R3, R4, R5, R6: footprint (none) -> Resistor_SMD:R_0402_1005Metric_Pad0.72x0.64mm_HandSolder
Connections:
- net GND: now also J3.2
- net VCC: now also J3.1
Other:
- note added: "4.5-14 V DC"
- note added: "Line Level"
- note added: "Power Input"

Commit message: Layout improvements for amp
Parts:
- J1: footprint Connector_Audio:Jack_3.5mm_CUI_SJ1-3525N_Horizontal -> Connector_Audio:Jack_3.5mm_CUI_SJ-3523-SMT_Horizontal
- L1, L2: footprint Capacitor_SMD:C_0402_1005Metric_Pad0.74x0.62mm_HandSolder -> Inductor_SMD:L_Taiyo-Yuden_MD-3030
Changed lines of the file:
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@@
       (effects (font (size 1.27 1.27)))
     )
-    (property "Footprint" "Capacitor_SMD:C_0402_1005Metric_Pad0.74x0.62mm_HandSolder" (at 198.755 104.14 0)
+    (property "Footprint" "Inductor_SMD:L_Taiyo-Yuden_MD-3030" (at 198.755 104.14 0)
       (effects (font (size 1.27 1.27)) hide)
     )
@@
       (effects (font (size 1.27 1.27)))
     )
-    (property "Footprint" "Connector_Audio:Jack_3.5mm_CUI_SJ1-3525N_Horizontal" (at 81.28 36.195 0)
+    (property "Footprint" "Connector_Audio:Jack_3.5mm_CUI_SJ-3523-SMT_Horizontal" (at 81.28 36.195 0)
       (effects (font (size 1.27 1.27)) hide)
     )
@@
       (effects (font (size 1.27 1.27)))
     )
-    (property "Footprint" "Capacitor_SMD:C_0402_1005Metric_Pad0.74x0.62mm_HandSolder" (at 198.755 85.09 0)
-      (effects (font (size 1.27 1.27)) hide)
-    )
+    (property "Footprint" "Inductor_SMD:L_Taiyo-Yuden_MD-3030" (at 198.755 85.09 0)
+      (effects (font (size 1.27 1.27)) hide)
+    )
