File: Electrical Design/Modules/Filter.kicad_sch (KiCad schematic)
At the start: 0 parts

Commit message: Noise Filter schematic with component Values
Parts:
- added C22: 0.1mF, symbol Device:C
- added R38: 1k, symbol Device:R
Connections:
- new net GND: C22.2
- new net Input: R38.1
- new net Output: C22.1, R38.2
