File: Electrical Design/PedalSynth/PedalSynth.kicad_sch (KiCad schematic)
At the start: 26 parts, among them J1 AudioJack3, J2 speakON_NL2MDXX-V, J3 Barrel_Jack, U1 TPA3136D2PWPR

Commit message: add kicad corner
Parts:
- C1, C2: footprint Capacitor_SMD:C_0805_2012Metric_Pad1.18x1.45mm_HandSolder -> Capacitor_THT:CP_Radial_D10.0mm_P5.00mm_P7.50mm
Connections:
- net GND: no longer C1.1, C2.1, C3.2, C4.1, C5.1, C6.2, C7.1, C9.2, J3.1, R1.1, R2.1, R4.2, U1.15 (PVCCR), U1.16 (PVCCR), U1.27 (PVCCL), U1.28 (PVCCL), U1.7 (AVCC), U1.9 (GVDD)
- net /SHUTDOWN: no longer R2.2, R3.2, R4.1, U1.10 (PLIMIT), U1.14 (PBTL)
- removed net OFILTER: C11.1, C11.2, C12.1, C12.2, L1.1, L2.1, U1.17 (BSPR), U1.18 (OUTPR), U1.20 (OUTNR), U1.21 (BSNR), U1.22 (BSNL), U1.23 (OUTNL), U1.25 (OUTPL), U1.26 (BSPL)
- net SPKR renamed SPK+
- net SPK+: no longer C14.1, J2.1-, L2.2
- new net: R2.2, U1.14 (PBTL)
- new net: R3.2, R4.1, U1.10 (PLIMIT)
- new net BSNR: C12.1, U1.17 (BSPR), U1.21 (BSNR)
- new net BSPL: C11.1, U1.22 (BSNL), U1.26 (BSPL)
- new net GVDD: C9.2, R4.2, U1.9 (GVDD)
- new net OUTPL: C11.2, L1.1, U1.23 (OUTNL), U1.25 (OUTPL)
- new net OUTPR: C12.2, L2.1, U1.18 (OUTPR), U1.20 (OUTNR)
- new net SPK-: C14.1, J2.1-, L2.2
- new net VCC: C1.1, C2.1, C3.2, C4.1, C5.1, C6.2, C7.1, J3.1, R1.1, R2.1, U1.15 (PVCCR), U1.16 (PVCCR), U1.27 (PVCCL), U1.28 (PVCCL), U1.7 (AVCC)
Other:
- moved on the sheet: C1

Commit message: update to v8
Parts:
- removed R4: 56k, Resistor_SMD:R_0402_1005Metric_Pad0.72x0.64mm_HandSolder, symbol Device:R
- added RV1: 100k, Potentiometer_THT:Potentiometer_Bourns_3386P_Vertical, symbol Device:R_Potentiometer
- added TP1, TP2: TestPoint, TestPoint:TestPoint_Bridge_Pitch2.0mm_Drill0.7mm, symbol Connector:TestPoint
- C1, C2: footprint Capacitor_THT:CP_Radial_D10.0mm_P5.00mm_P7.50mm -> Capacitor_THT:CP_Radial_D8.0mm_P3.50mm
- L1, L2: footprint Inductor_SMD:L_Taiyo-Yuden_MD-3030 -> HC9-330-R:IND_COILECTRONICS_HC9_B-M
- R3: value 39k -> 10k
Connections:
- net GVDD: now also RV1.1
- net SPK+: now also TP1.1
- net SPK-: now also TP2.1
- net at U1.10 (PLIMIT): now also RV1.2; no longer R3.2
- new net: R3.2, RV1.3
Other:
- moved on the sheet: R3

Commit message: update amp schematic and pcb
Parts:
- L1, L2: footprint HC9-330-R:IND_COILECTRONICS_HC9_B-M -> VLS6045AF_330M:IND_VLS6045AF-330M
Changed lines of the file:
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@@
 			)
 		)
-		(property "Footprint" "HC9-330-R:IND_COILECTRONICS_HC9_B-M"
+		(property "Footprint" "VLS6045AF_330M:IND_VLS6045AF-330M"
 			(at 198.755 104.14 0)
 			(effects
@@
 			)
 		)
-		(property "Footprint" "HC9-330-R:IND_COILECTRONICS_HC9_B-M"
+		(property "Footprint" "VLS6045AF_330M:IND_VLS6045AF-330M"
 			(at 198.755 85.09 0)
 			(effects

Commit message: r1.0 amp pcb
Parts:
- added GND1, RING1, SLEEVE1: TestPoint, TestPoint:TestPoint_Bridge_Pitch2.0mm_Drill0.7mm, symbol Connector:TestPoint
- J2: value speakON_NL2MDXX-V -> Pheonix Latching Connector (1190297); footprint Connector_Audio:Jack_speakON_Neutrik_NL2MDXX-H-3_Horizontal -> Pheonix-2P-Level1190297:PHOENIX_1190297; symbol Connector_Audio:SpeakON_NL2 -> Pheonix-1190297:1190297; MANUFACTURER (none) -> Phoenix Contact; MAXIMUM_PACKAGE_HEIGHT (none) -> 23.58mm; PARTREV (none) -> 03.11.2020; STANDARD (none) -> Manufacturer Recommendations
- J3: footprint Connector_BarrelJack:BarrelJack_CUI_PJ-063AH_Horizontal -> Connector_BarrelJack:BarrelJack_Wuerth_6941xx301002
- L1, L2: footprint VLS6045AF_330M:IND_VLS6045AF-330M -> Inductor-VLS6045AF_330M:IND_VLS6045AF-330M
- renumbered TP1 to TPSP1, TP2 to TPSP2
Connections:
- net GND: now also GND1.1
- net SPK+: now also J2.2_1, J2.2_2; no longer J2.1+
- net SPK-: now also J2.1_1, J2.1_2; no longer J2.1-
- net at J1.T, R6.1: now also SLEEVE1.1
- net at J1.R, R5.2: now also RING1.1

Commit message: amp changes
Parts:
- C11, C12: value .47u -> .27u
Changed lines of the file:
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@@
 			)
 		)
-		(property "Value" ".47u"
+		(property "Value" ".27u"
 			(at 184.785 101.6 90)
 			(effects
@@
 			)
 		)
-		(property "Value" ".47u"
+		(property "Value" ".27u"
 			(at 184.785 107.95 90)
 			(effects
