File: Electrical Design/Modules/ECE 411 Project/ECE 411 Project.kicad_pcb (KiCad board)
At the start: 2 copper layers, 120 parts, among them J1 5mm 9V Barrel, J2 BOOST, Q1 NPN, Q2 2N3904, Q3 2N3904, Q4 2N3904, Q5 PNP, Q6 PNP, SW1 SW_Push, SW2 SW_Push, SW3 SW_Push, SW4 SW_Push, SW5 SW_Push, SW6 SW_Push, SW7 SW_Push, SW8 SW_Push, U1 HT7333, U11 ESP32-WROOM-32, U2 LT1054, U3 MN3207, U7 TL072, U9 TPA3136D2PWPR

Commit message: export pdfs
Parts:
- moved U7 155.3 mm to (51.9, 112.0), turned to 90 degrees
- moved C3 144.8 mm to (73.9, 99.4)
- moved C33 142.5 mm to (106.4, 121.0)
- moved C34 142.5 mm to (106.4, 123.0)
- moved C35 142.5 mm to (106.4, 124.9)
- moved C29 139.3 mm to (111.4, 122.0)
- moved C30 139.3 mm to (111.4, 124.0)
- moved C31 139.3 mm to (111.4, 125.9)
- moved R1 139.0 mm to (64.6, 111.2), turned to 90 degrees
- moved Q1 138.6 mm to (67.2, 106.1), turned to 90 degrees
- moved C25 138.4 mm to (89.5, 119.2)
- moved C26 138.4 mm to (98.4, 106.4)
- moved C27 138.4 mm to (98.4, 109.4)
- moved C28 138.4 mm to (98.4, 112.4)
- moved C32 138.4 mm to (98.4, 115.4)
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Other:
- board outline added: 99 x 99 mm
- board text added: "PedalSynth b1.0 7 November 2024"

Commit message: update kicad
Parts:
- added D3: LED, LED_THT:LED_D5.0mm, F.Cu at (146.5, 64.0)
- added J3: Pheonix Connector, 1190297:PHOENIX_1190297, F.Cu at (114.3, 68.7)
- added RV3: 10k, Connector_PinSocket_2.54mm:PinSocket_1x03_P2.54mm_Vertical, F.Cu at (128.9, 52.9)
- added RV6: 100k, Connector_PinSocket_2.54mm:PinSocket_1x03_P2.54mm_Vertical, F.Cu at (146.3, 52.9)
- added U4: NE555D, Package_SO:SOIC-8_3.9x4.9mm_P1.27mm, F.Cu at (137.4, 65.6)
- added U5: LTV-827, Package_DIP:DIP-8_W7.62mm, F.Cu at (134.8, 52.6)
- C2: value 10nF -> 4.7uF
- R1: value 1M -> 1.2k
- R2: value 10k -> 1.2k
- RV2: value Depth 5k -> 10k
Connections:
- C2 pad 1: Net-(U7A-+) -> GND
- C2 pad 2: Net-(C2-Pad2) -> Net-(U4-THR)
- C23 pad 1: /Chorus Effect/CHORUSOUT -> /Class-D Amplification/AMPIN
- C31 pad 2: /Chorus Effect/CHORUSOUT -> /Class-D Amplification/AMPIN
- R1 pad 1: /Chorus Effect/CHORUSOUT -> +9V
- R1 pad 2: GND -> Net-(U4-DIS)
- R2 pad 1: Net-(Q1-B) -> /Chorus Effect/CLK
- RV1 pad 1: Net-(C3-Pad1) -> /ESP32-S3-WROOM/GENOUT
- RV1 pad 2: Net-(C2-Pad2) -> /Chorus Effect/CHORUSIN
- RV1 pad 3: Net-(C2-Pad2) -> unconnected-(RV1-Pad3)
- RV2 pad 1: Net-(R11-Pad1) -> /Chorus Effect/CHORUSIN
- RV2 pad 2: Net-(C3-Pad2) -> /Chorus Effect/CHORUSOUT
- RV2 pad 3: Net-(R2-Pad2) -> unconnected-(RV2-Pad3)
- U11 pad 30: /Chorus Effect/CLK -> /ESP32-S3-WROOM/CLK

Commit message: PCB V2!!!
Parts:
- removed C3: 10uF, Capacitor_SMD:C_1210_3225Metric_Pad1.33x2.70mm_HandSolder
- removed C9: 10uF, Capacitor_SMD:C_1206_3216Metric_Pad1.33x1.80mm_HandSolder
- removed Q1: NPN, Package_TO_SOT_THT:TO-52-3
- removed R11: 1k, Resistor_SMD:R_0805_2012Metric_Pad1.20x1.40mm_HandSolder
- removed R12, R13, R14, R15: 220k, Resistor_SMD:R_0805_2012Metric_Pad1.20x1.40mm_HandSolder
- removed TPSP1, TPSP2: TestPoint, TestPoint:TestPoint_Bridge_Pitch2.0mm_Drill0.7mm
- removed U11: ESP32-WROOM-32, RF_Module:ESP32-WROOM-32
- removed U7: TL072, Package_DIP:CERDIP-8_W7.62mm_SideBrazed
- added CHO-TRE1: TestPoint, TestPoint:TestPoint_THTPad_2.5x2.5mm_Drill1.2mm, F.Cu at (116.6, 80.2)
- added CLK1: TestPoint, TestPoint:TestPoint_THTPad_2.5x2.5mm_Drill1.2mm, F.Cu at (88.0, 67.6)
- added FUZ-CHO1: TestPoint, TestPoint:TestPoint_THTPad_2.5x2.5mm_Drill1.2mm, F.Cu at (126.7, 37.4)
- added J4: 1/8in Jack, Connector_Audio:Jack_3.5mm_CUI_SJ-3523-SMT_Horizontal, F.Cu at (38.2, 65.3)
- added J5: 1/4in Jack, Connector_PinSocket_2.54mm:PinSocket_1x02_P2.54mm_Vertical, F.Cu at (83.5, 108.5)
- added OUT_{LINE}1: TestPoint, TestPoint:TestPoint_THTPad_2.5x2.5mm_Drill1.2mm, F.Cu at (65.6, 96.2)
- added RV7: 10k, Connector_PinSocket_2.54mm:PinSocket_1x03_P2.54mm_Vertical, F.Cu at (70.0, 103.0)
- added SPK+1: TestPoint, TestPoint:TestPoint_Bridge_Pitch2.0mm_Drill0.7mm, F.Cu at (42.5, 118.0)
- added SPK-1: TestPoint, TestPoint:TestPoint_Bridge_Pitch2.0mm_Drill0.7mm, F.Cu at (42.5, 99.0)
- added SW9: SW_SPDT, Button_Switch_THT:SW_Slide_SPDT_Angled_CK_OS102011MA1Q, F.Cu at (35.0, 75.0)
- added U6: ~, Module:PinHeader_ESP32_WROOM_Narrow, F.Cu at (52.6, 42.0)
- added V4.5: TestPoint, TestPoint:TestPoint_THTPad_2.5x2.5mm_Drill1.2mm, F.Cu at (78.2, 77.0)
- added V9: TestPoint, TestPoint:TestPoint_THTPad_2.5x2.5mm_Drill1.2mm, F.Cu at (52.2, 82.0)
- added VGND1: TestPoint, TestPoint:TestPoint_THTPad_2.5x2.5mm_Drill1.2mm, F.Cu at (36.6, 98.2)
- C1: value 0.047uF -> 47nF
- C11: value 0.068uF -> 68nF
- C13, C41: value 0.0033uF -> 3.3nF
- C14, C17: value 0.0082uF -> 8.2nF
- C16: value 0.033u -> 33nF
- C19: value 0.033uF -> 33nF
- C2, C6: footprint Capacitor_SMD:C_0805_2012Metric_Pad1.18x1.45mm_HandSolder -> Capacitor_SMD:C_1206_3216Metric_Pad1.33x1.80mm_HandSolder
- C20: value 0.0068uF -> 6.8nF
- C23: value 0.1mF -> 1uF
- C24, C25: value 100u -> 100uF
- C26, C27: value .1u -> .1uF
- C28, C32, C36, C37: value 1u -> 1uF
- C29, C30: footprint Capacitor_SMD:C_0402_1005Metric_Pad0.74x0.62mm_HandSolder -> Capacitor_SMD:C_0805_2012Metric_Pad1.18x1.45mm_HandSolder
- C31: value 0.1u -> 0.1uF; footprint Capacitor_SMD:C_0402_1005Metric_Pad0.74x0.62mm_HandSolder -> Capacitor_SMD:C_0805_2012Metric_Pad1.18x1.45mm_HandSolder
- C33: value .27u -> .1uF; footprint Capacitor_SMD:C_0402_1005Metric_Pad0.74x0.62mm_HandSolder -> Capacitor_SMD:C_0805_2012Metric_Pad1.18x1.45mm_HandSolder
- C34: value .47u -> .47uF; footprint Capacitor_SMD:C_0402_1005Metric_Pad0.74x0.62mm_HandSolder -> Capacitor_SMD:C_0805_2012Metric_Pad1.18x1.45mm_HandSolder
- C35: value .47u -> .47uf; footprint Capacitor_SMD:C_0402_1005Metric_Pad0.74x0.62mm_HandSolder -> Capacitor_SMD:C_0805_2012Metric_Pad1.18x1.45mm_HandSolder
- C39: value 0.01uF -> 10nF
- C4: footprint Capacitor_SMD:C_1812_4532Metric_Pad1.57x3.40mm_HandSolder -> Capacitor_SMD:C_1206_3216Metric_Pad1.33x1.80mm_HandSolder
- C40: value 20uF -> 22uF
- C42: footprint Capacitor_THT:CP_Radial_D6.3mm_P2.50mm -> Capacitor_THT:CP_Radial_D8.0mm_P3.50mm
- C7: value 100nF -> 0.1uF
- J2: footprint Connector_PinHeader_2.54mm:PinHeader_1x02_P2.54mm_Horizontal -> Connector_PinHeader_2.54mm:PinHeader_1x02_P2.54mm_Vertical
- L1, L2: value 33u -> 33uF
- OLED1: value ~ -> OLED-I2C
- R40, R43: footprint Resistor_SMD:R_0402_1005Metric_Pad0.72x0.64mm_HandSolder -> Resistor_SMD:R_0805_2012Metric_Pad1.20x1.40mm_HandSolder
- RV1, RV2: footprint Connector_PinHeader_2.54mm:PinHeader_1x03_P2.54mm_Vertical -> Connector_PinSocket_2.54mm:PinSocket_1x03_P2.54mm_Vertical
- moved J3 89.0 mm to (32.5, 103.9), turned to -90 degrees
- moved GND1 86.6 mm to (36.0, 118.0)
- moved RV1 81.8 mm to (103.9, 36.0), turned to 90 degrees
- moved RV6 77.7 mm to (87.4, 103.5)
- moved D3 60.2 mm to (98.3, 100.0)
- moved L1 59.9 mm to (54.7, 117.4), turned to 180 degrees
- moved L2 59.4 mm to (55.0, 109.7), turned to 180 degrees
- moved U4 58.1 mm to (92.2, 102.2), turned to -90 degrees
- moved U5 55.7 mm to (98.4, 94.8), turned to 90 degrees
- moved RV2 54.3 mm to (110.2, 77.9), turned to 0 degrees
- moved SW1 50.7 mm to (80.5, 59.0), turned to -90 degrees
- moved R43 49.5 mm to (73.7, 108.5), turned to 180 degrees
- moved C37 47.8 mm to (53.5, 105.0)
- moved R40 47.2 mm to (75.0, 122.5), turned to 90 degrees
- moved C35 46.2 mm to (62.1, 112.0), turned to -90 degrees
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Connections:
- net /ESP32-S3-WROOM/GENOUT renamed /ESP32-S3-WROOM Dev Board/GENOUT
- C23 pad 1: /Class-D Amplification/AMPIN -> /LineOut
- C24 pad 1: VCC -> Vin
- C25 pad 1: VCC -> Vin
- C26 pad 2: VCC -> Vin
- C27 pad 1: VCC -> Vin
- C28 pad 1: +9V -> Vin
- C29 pad 2: VCC -> Vin
- C30 pad 1: VCC -> Vin
- C31 pad 2: /Class-D Amplification/AMPIN -> /LineOut
- C4 pad 1: Net-(D1-A) -> Vin
- C42 pad 1: Net-(D1-A) -> Vin
- C43 pad 2: Net-(D1-A) -> Vin
- D1 pad 2: Net-(D1-A) -> Vin
- J1 pad 1: Net-(D1-A) -> Vin
- J3 pad 1_1: /Class-D Amplification/SPK+ -> /Class-D Amplification/SPK-
- J3 pad 1_2: /Class-D Amplification/SPK+ -> /Class-D Amplification/SPK-
- J3 pad 2_1: /Class-D Amplification/SPK- -> /Class-D Amplification/SPK+
- J3 pad 2_2: /Class-D Amplification/SPK- -> /Class-D Amplification/SPK+
- OLED1 pad 3: /ESP32-S3-WROOM/SDA -> /ESP32-S3-WROOM Dev Board/SDA
- OLED1 pad 4: /ESP32-S3-WROOM/SCL -> /ESP32-S3-WROOM Dev Board/SCL
- Q5 pad 3: unconnected-(Q5-E-Pad3) -> GND
- R40 pad 1: VCC -> Vin
- R43 pad 1: +9V -> Vin
- RV3 pad 2: /Class-D Amplification/AMPIN -> /Tremolo Effect/TREMOUT
- SW1 pad 2: /ESP32-S3-WROOM/BTN0 -> /ESP32-S3-WROOM Dev Board/BTN0
- SW2 pad 2: /ESP32-S3-WROOM/BTN1 -> /ESP32-S3-WROOM Dev Board/BTN1
- SW3 pad 2: /ESP32-S3-WROOM/BTN2 -> /ESP32-S3-WROOM Dev Board/BTN2
- SW4 pad 2: /ESP32-S3-WROOM/BTN3 -> /ESP32-S3-WROOM Dev Board/BTN3
- SW5 pad 2: /ESP32-S3-WROOM/BTN4 -> /ESP32-S3-WROOM Dev Board/BTN4
- SW6 pad 2: /ESP32-S3-WROOM/BTN5 -> /ESP32-S3-WROOM Dev Board/BTN5
- SW7 pad 2: /ESP32-S3-WROOM/BTN6 -> /ESP32-S3-WROOM Dev Board/BTN6
- SW8 pad 2: /ESP32-S3-WROOM/BTN7 -> /ESP32-S3-WROOM Dev Board/BTN7
- U1 pad 2: Net-(D1-A) -> Vin
- U5 pad 7: /Class-D Amplification/AMPIN -> /Tremolo Effect/TREMOUT
- U9 pad 15: VCC -> Vin
- U9 pad 16: VCC -> Vin
- U9 pad 27: VCC -> Vin
- U9 pad 28: VCC -> Vin
- U9 pad 7: +9V -> Vin
Routing:
- net +9V: track 8.94 -> 217.8 mm, vias 0 -> 5
- net Vin: track 0.00 -> 130.9 mm, vias 0 -> 8
- net +5V: track 9.36 -> 118.3 mm, vias 0 -> 3
- net +4.5V: track 4.41 -> 104.1 mm, vias 0 -> 6
- net /ESP32-S3-WROOM Dev Board/GENOUT: track 0.00 -> 83.6 mm, vias 0 -> 2
- net /Chorus Effect/CHORUSIN: track 0.00 -> 79.9 mm
- net /Tremolo Effect/TREMOUT: track 0.00 -> 66.2 mm
- net /ESP32-S3-WROOM Dev Board/SDA: track 0.00 -> 54.8 mm
- net Net-(U3-IN): track 0.00 -> 53.0 mm
- net /ESP32-S3-WROOM Dev Board/SCL: track 0.00 -> 52.3 mm
- net Net-(V3207D2-+): track 0.00 -> 41.8 mm
- net /ESP32-S3-WROOM Dev Board/BTN7: track 0.00 -> 36.5 mm
- net Net-(C12-Pad1): track 0.00 -> 34.8 mm
- net -9V: track 37.8 -> 70.4 mm, vias 0 -> 4
- net /Class-D Amplification/SPK-: track 0.00 -> 31.3 mm
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Other:
- board text added: "SynthBuddy r1.0 14 November 2024"
- board text removed: "PedalSynth b1.0 7 November 2024"

Commit message: DRAFT PACKAGE
Parts:
- added ?: , clipboard:cb89ceac-0acd-432b-9393-97274f22b4f5, F.Cu at (126.3, 109.7)
- moved R32 0.71 mm to (88.5, 77.9)
Routing:
- net /Tremolo Effect/TREMOUT: track 66.2 -> 102.9 mm, vias 0 -> 1
- net /Chorus Effect/CHORUSOUT: track 30.7 -> 51.5 mm, vias 0 -> 2
- net Net-(V3207D2-+): track 41.8 -> 59.3 mm, vias 0 -> 2
- net Net-(U4-THR): track 5.48 -> 21.7 mm, vias 0 -> 2
- net +9V: track 217.8 -> 232.4 mm
- net Net-(R34-Pad2): track 2.88 -> 8.77 mm
- net Net-(U4-DIS): track 6.58 -> 12.4 mm
Other:
- board size 99 x 99 mm -> 99.2 x 99.2 mm
- board text added: "SynthBuddy"
- board text added: "r1.1 14 November 2024"
- board text removed: "SynthBuddy r1.0 14 November 2024"
