File: Electrical Design/Modules/ECE 411 Project/ECE 411 Project.kicad_sch (KiCad schematic)
At the start: 42 parts, among them J1 5mm 9V Barrel, J2 BOOST, J3 Pheonix Connector, J4 1/8in Jack, J5 1/4in Jack, SW1 SW_Push, SW2 SW_Push, SW3 SW_Push, SW4 SW_Push, SW5 SW_Push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

Commit message: schematic changes
Other:
- sheet ESP32-S3-WROOM Dev Board ports: added none; removed CLK
- note added: "OLED Readout"
- moved on the sheet: OLED1
Changed lines of the file:
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@@
 	(wire
 		(pts
-			(xy 73.66 22.225) (xy 73.66 36.195)
+			(xy 81.28 21.59) (xy 81.28 32.385)
 		)
 		(stroke
@@
 	(wire
 		(pts
-			(xy 73.66 36.195) (xy 78.74 36.195)
+			(xy 81.28 32.385) (xy 86.36 32.385)
 		)
 		(stroke
@@
 	(wire
 		(pts
-			(xy 98.425 19.05) (xy 98.425 22.225)
+			(xy 106.045 19.685) (xy 106.045 21.59)
 		)
 		(stroke
@@
 	(wire
 		(pts
-			(xy 70.485 38.735) (xy 78.74 38.735)
+			(xy 70.485 34.925) (xy 86.36 34.925)
 		)
 		(stroke
@@
 	(wire
 		(pts
-			(xy 75.565 24.13) (xy 98.425 24.13)
+			(xy 83.185 23.495) (xy 106.045 23.495)
 		)
 		(stroke
@@
 	(wire
 		(pts
-			(xy 98.425 24.13) (xy 98.425 27.305)
+			(xy 106.045 23.495) (xy 106.045 26.67)
 		)
 		(stroke
@@
 	(wire
 		(pts
-			(xy 75.565 33.655) (xy 75.565 24.13)
+			(xy 83.185 29.845) (xy 83.185 23.495)
 		)
 		(stroke
@@
 	(wire
 		(pts
-			(xy 78.74 33.655) (xy 75.565 33.655)
+			(xy 86.36 29.845) (xy 83.185 29.845)
 		)
 		(stroke
@@
 	(wire
 		(pts
-			(xy 70.485 41.275) (xy 78.74 41.275)
+			(xy 70.485 37.465) (xy 86.36 37.465)
 		)
 		(stroke
@@
 	(wire
 		(pts
-			(xy 98.425 22.225) (xy 73.66 22.225)
+			(xy 106.045 21.59) (xy 81.28 21.59)
 		)
 		(stroke
@@
 	)
 	(rectangle
+		(start 78.105 12.7)
+		(end 113.665 41.275)
+		(stroke
+			(width 0)
+			(type dash)
+			(color 72 72 72 1)
+		)
+		(fill
+			(type none)
+		)
+	)
+	(rectangle
 		(start 257.175 52.07)
 		(end 283.21 74.93)
@@
 		)
 	)
+	(text "OLED Readout"
+		(exclude_from_sim no)
+		(at 106.045 43.18 0)
+		(effects
+			(font
+				(size 1.5 1.5)
+				(thickness 0.254)
+				(bold yes)
+			)
+		)
+	)
 	(text "Wave & Frequency Select"
 		(exclude_from_sim no)
@@
 	(global_label "+5V"
 		(shape output)
-		(at 98.425 19.05 90)
+		(at 106.045 19.685 90)
 		(fields_autoplaced yes)
 		(effects
@@
 		)
 		(property "Intersheetrefs" "${INTERSHEET_REFS}"
-			(at 98.425 12.1943 90)
+			(at 106.045 12.8293 90)
 			(effects
 				(font
@@
 	(symbol
 		(lib_id "Project Specific Library:OLED_SSD1306")
-		(at 86.36 29.845 0)
+		(at 93.98 26.035 0)
 		(unit 1)
 		(exclude_from_sim no)
@@
 		(dnp no)
 		(property "Reference" "OLED1"
-			(at 81.28 29.845 0)
+			(at 88.9 26.035 0)
 			(effects
 				(font
@@
 		)
 		(property "Value" "OLED-I2C"
-			(at 93.345 38.735 0)
+			(at 100.965 34.925 0)
 			(effects
 				(font
@@
 		)
 		(property "Footprint" "Connector_PinHeader_2.54mm:PinHeader_1x04_P2.54mm_Vertical"
-			(at 86.36 29.845 0)
+			(at 93.98 26.035 0)
 			(effects
 				(font
@@
 		)
 		(property "Datasheet" "https://www.mouser.com/datasheet/2/1398/Soldered_333099-3395096.pdf"
-			(at 86.36 29.845 0)
+			(at 93.98 26.035 0)
 			(effects
 				(font
@@
 		)
 		(property "Description" ""
-			(at 86.36 29.845 0)
+			(at 93.98 26.035 0)
 			(effects
 				(font
@@
 		)
 		(property "Part Number" ""
-			(at 86.36 29.845 0)
+			(at 93.98 26.035 0)
 			(effects
 				(font
@@
 		)
 		(property "Part Origin" ""
-			(at 86.36 29.845 0)
+			(at 93.98 26.035 0)
 			(effects
 				(font
@@
 		)
 		(property "On Hand (On Way)" ""
-			(at 86.36 29.845 0)
+			(at 93.98 26.035 0)
 			(effects
 				(font
@@
 	(symbol
 		(lib_id "power:GND")
-		(at 98.425 27.305 0)
+		(at 106.045 26.67 0)
 		(unit 1)
 		(exclude_from_sim no)
@@
 		(fields_autoplaced yes)
 		(property "Reference" "#PWR06"
-			(at 98.425 33.655 0)
+			(at 106.045 33.02 0)
 			(effects
 				(font
@@
 		)
 		(property "Value" "GND"
-			(at 98.425 31.75 0)
+			(at 106.045 31.115 0)
 			(effects
 				(font
@@
 		)
 		(property "Footprint" ""
-			(at 98.425 27.305 0)
+			(at 106.045 26.67 0)
 			(effects
 				(font
@@
 		)
 		(property "Datasheet" ""
-			(at 98.425 27.305 0)
+			(at 106.045 26.67 0)
 			(effects
 				(font
@@
 		)
 		(property "Description" "Power symbol creates a global label with name \"GND\" , ground"
-			(at 98.425 27.305 0)
+			(at 106.045 26.67 0)
 			(effects
 				(font
@@
 		)
 		(pin "SDA" bidirectional
-			(at 70.485 38.735 0)
+			(at 70.485 34.925 0)
 			(effects
 				(font
@@
 		)
 		(pin "SCL" bidirectional
-			(at 70.485 41.275 0)
-			(effects
-				(font
-					(size 1.27 1.27)
-				)
-				(justify right)
-			)
-		)
-		(pin "CLK" output
-			(at 70.485 52.07 0)
+			(at 70.485 37.465 0)
 			(effects
 				(font

Commit message: schematic update
Other:
- title: PedalSynth PWM Synthesizer -> SynthBuddy
Changed lines of the file:
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@@
 	(paper "A4")
 	(title_block
-		(title "PedalSynth PWM Synthesizer")
+		(title "SynthBuddy")
 		(date "2024-11-14")
-		(rev "r2.0")
+		(rev "r2.1")
 		(company "Portland State University")
 		(comment 1 "Open Source Hardware")
