File: Electrical Design/Modules/ECE 411 Project/Amp.kicad_sch (KiCad schematic)
At the start: 22 parts, among them U9 TPA3136D2PWPR

Commit message: bom changes
Parts:
- renumbered TPSP1 to SPK+, TPSP2 to SPK-
Changed lines of the file:
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@@
 		)
 		(instances
-			(project "ECE 411 Project"
+			(project ""
 				(path "/2625e5a1-d0c8-41ce-941d-75d035a5f1c5/fc48e9dd-306b-4a9b-831b-312573108cdc"
 					(reference "#PWR030")
@@
 		(on_board yes)
 		(dnp no)
-		(property "Reference" "TPSP2"
+		(property "Reference" "SPK-"
 			(at 194.945 98.425 0)
 			(effects
@@
 			(project "ECE 411 Project"
 				(path "/2625e5a1-d0c8-41ce-941d-75d035a5f1c5/fc48e9dd-306b-4a9b-831b-312573108cdc"
-					(reference "TPSP2")
+					(reference "SPK-")
 					(unit 1)
 				)
@@
 		(on_board yes)
 		(dnp no)
-		(property "Reference" "TPSP1"
+		(property "Reference" "SPK+"
 			(at 198.755 80.01 0)
 			(effects
@@
 			(project "ECE 411 Project"
 				(path "/2625e5a1-d0c8-41ce-941d-75d035a5f1c5/fc48e9dd-306b-4a9b-831b-312573108cdc"
-					(reference "TPSP1")
-					(unit 1)
-				)
+					(reference "SPK+")
+					(unit 1)
+				)

Commit message: update kicad
Parts:
- C24, C25: value 100u -> 100uF
- C26, C27: value .1u -> .1uF
- C28, C32, C36, C37: value 1u -> 1uF
- C31: value 0.1u -> 0.1uF
- C33: value .27u -> .1uF
- C34: value .47u -> .47uF
- C35: value .47u -> .47uf
- L1, L2: value 33u -> 33uF
Changed lines of the file:
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@@
 	(title_block
 		(title "20W Mono Class-D Audio Amplifier")
-		(date "2024-11-07")
-		(rev "2.5")
+		(date "2024-11-13")
+		(rev "2.6")
 		(company "Portland State University")
 		(comment 1 "Open Source Hardware")
@@
 			)
 		)
-		(property "Value" "100u"
+		(property "Value" "100uF"
 			(at 83.82 78.74 0)
 			(effects
@@
 			)
 		)
-		(property "Value" "1u"
+		(property "Value" "1uF"
 			(at 210.185 92.71 0)
 			(effects
@@
 		(fields_autoplaced yes)
 		(property "Reference" "C33"
-			(at 122.555 112.395 0)
+			(at 129.54 112.3949 0)
 			(effects
 				(font
 					(size 1.27 1.27)
 				)
-				(justify right)
+				(justify left)
 			)
 		)
-		(property "Value" ".27u"
-			(at 122.555 114.935 0)
+		(property "Value" ".1uF"
+			(at 129.54 114.9349 0)
 			(effects
 				(font
 					(size 1.27 1.27)
 				)
-				(justify right)
+				(justify left)
 			)
 		)
@@
 			)
 		)
-		(property "Value" "100u"
+		(property "Value" "100uF"
 			(at 80.01 101.6 0)
 			(effects
@@
 			)
 		)
-		(property "Value" ".47u"
+		(property "Value" ".47uf"
 			(at 179.07 109.22 90)
 			(effects
@@
 			)
 		)
-		(property "Value" ".1u"
+		(property "Value" ".1uF"
 			(at 88.265 101.6 0)
 			(effects
@@
 			)
 		)
-		(property "Value" "33u"
+		(property "Value" "33uF"
 			(at 193.04 102.235 90)
 			(effects
@@
 			)
 		)
-		(property "Value" "1u"
+		(property "Value" "1uF"
 			(at 88.265 71.12 0)
 			(effects
@@
 			)
 		)
-		(property "Value" "1u"
+		(property "Value" "1uF"
 			(at 127.635 80.01 0)
 			(effects
@@
 			)
 		)
-		(property "Value" ".47u"
+		(property "Value" ".47uF"
 			(at 179.07 102.87 90)
 			(effects
@@
 			)
 		)
-		(property "Value" ".1u"
+		(property "Value" ".1uF"
 			(at 88.265 79.375 0)
 			(effects
@@
 			)
 		)
-		(property "Value" "33u"
+		(property "Value" "33uF"
 			(at 193.04 83.185 90)
 			(effects
@@
 			)
 		)
-		(property "Value" "1u"
+		(property "Value" "1uF"
 			(at 210.185 110.49 0)
 			(effects
@@
 			)
 		)
-		(property "Value" "0.1u"
+		(property "Value" "0.1uF"
 			(at 106.68 113.665 90)
 			(effects

Commit message: add switch to schematic
Parts:
- renumbered SPK+ to SPK+1, SPK- to SPK-1
Changed lines of the file:
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@@
 		(on_board yes)
 		(dnp no)
-		(property "Reference" "SPK-"
+		(property "Reference" "SPK-1"
 			(at 194.945 98.425 0)
 			(effects
@@
 			(project "ECE 411 Project"
 				(path "/2625e5a1-d0c8-41ce-941d-75d035a5f1c5/fc48e9dd-306b-4a9b-831b-312573108cdc"
-					(reference "SPK-")
+					(reference "SPK-1")
 					(unit 1)
 				)
@@
 		(on_board yes)
 		(dnp no)
-		(property "Reference" "SPK+"
+		(property "Reference" "SPK+1"
 			(at 198.755 80.01 0)
 			(effects
@@
 			(project "ECE 411 Project"
 				(path "/2625e5a1-d0c8-41ce-941d-75d035a5f1c5/fc48e9dd-306b-4a9b-831b-312573108cdc"
-					(reference "SPK+")
-					(unit 1)
-				)
+					(reference "SPK+1")
+					(unit 1)
+				)

Commit message: PCB V2!!!
Connections:
- net VCC is gone; now on net Vin: C24.1, C25.1, C26.2, C27.1, C29.2, C30.1, R40.1, U9.15 (PVCCR), U9.16 (PVCCR), U9.27 (PVCCL), U9.28 (PVCCL)
Changed lines of the file:
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@@
+	(hierarchical_label "Vin"
+		(shape input)
+		(at 71.12 87.63 90)
+		(fields_autoplaced yes)
+		(effects
+			(font
+				(size 1.27 1.27)
+			)
+			(justify left)
+		)
+	)
+	(hierarchical_label "Vin"
+		(shape input)
+		(at 76.2 87.63 90)
+		(fields_autoplaced yes)
+		(effects
+			(font
+				(size 1.27 1.27)
+			)
+			(justify left)
+		)
+	)
 	(hierarchical_label "Vin"
 		(shape input)
@@
 		)
 	)
+	(hierarchical_label "Vin"
+		(shape input)
+		(at 87.63 118.745 90)
+		(fields_autoplaced yes)
+		(effects
+			(font
+				(size 1.27 1.27)
+			)
+			(justify left)
+		)
+	)
 	(hierarchical_label "{slash}SHUTDOWN"
 		(shape input)
@@
 	)
 	(symbol
-		(lib_name "VCC_1")
-		(lib_id "power:VCC")
-		(at 71.12 87.63 0)
-		(unit 1)
-		(exclude_from_sim no)
-		(in_bom yes)
-		(on_board yes)
-		(dnp no)
-		(fields_autoplaced yes)
-		(property "Reference" "#PWR026"
-			(at 71.12 91.44 0)
-			(effects
-				(font
-					(size 1.27 1.27)
-				)
-				(hide yes)
-			)
-		)
-		(property "Value" "VCC"
-			(at 71.12 83.185 0)
-			(effects
-				(font
-					(size 1.27 1.27)
-				)
-			)
-		)
-		(property "Footprint" ""
-			(at 71.12 87.63 0)
-			(effects
-				(font
-					(size 1.27 1.27)
-				)
-				(hide yes)
-			)
-		)
-		(property "Datasheet" ""
-			(at 71.12 87.63 0)
-			(effects
-				(font
-					(size 1.27 1.27)
-				)
-				(hide yes)
-			)
-		)
-		(property "Description" "Power symbol creates a global label with name \"VCC\""
-			(at 71.12 87.63 0)
-			(effects
-				(font
-					(size 1.27 1.27)
-				)
-				(hide yes)
-			)
-		)
-		(pin "1"
-		)
-		(instances
-			(project "ECE 411 Project"
-				(path "/2625e5a1-d0c8-41ce-941d-75d035a5f1c5/fc48e9dd-306b-4a9b-831b-312573108cdc"
-					(reference "#PWR026")
-					(unit 1)
-				)
-			)
-		)
-	)
-	(symbol
 		(lib_id "Device:C")
 		(at 206.375 91.44 0)
@@
 	)
 	(symbol
-		(lib_name "VCC_2")
-		(lib_id "power:VCC")
-		(at 76.2 87.63 0)
-		(unit 1)
-		(exclude_from_sim no)
-		(in_bom yes)
-		(on_board yes)
-		(dnp no)
-		(fields_autoplaced yes)
-		(property "Reference" "#PWR027"
-			(at 76.2 91.44 0)
-			(effects
-				(font
-					(size 1.27 1.27)
-				)
-				(hide yes)
-			)
-		)
-		(property "Value" "VCC"
-			(at 76.2 83.185 0)
-			(effects
-				(font
-					(size 1.27 1.27)
-				)
-			)
-		)
-		(property "Footprint" ""
-			(at 76.2 87.63 0)
-			(effects
-				(font
-					(size 1.27 1.27)
-				)
-				(hide yes)
-			)
-		)
-		(property "Datasheet" ""
-			(at 76.2 87.63 0)
-			(effects
-				(font
-					(size 1.27 1.27)
-				)
-				(hide yes)
-			)
-		)
-		(property "Description" "Power symbol creates a global label with name \"VCC\""
-			(at 76.2 87.63 0)
-			(effects
-				(font
-					(size 1.27 1.27)
-				)
-				(hide yes)
-			)
-		)
-		(pin "1"
-		)
-		(instances
-			(project "ECE 411 Project"
-				(path "/2625e5a1-d0c8-41ce-941d-75d035a5f1c5/fc48e9dd-306b-4a9b-831b-312573108cdc"
-					(reference "#PWR027")
-					(unit 1)
-				)
-			)
-		)
-	)
-	(symbol
 		(lib_name "PWR_FLAG_1")
 		(lib_id "power:PWR_FLAG")
@@
 					(unit 1)
 				)
-			)
-		)
-	)
-	(symbol
-		(lib_name "VCC_5")
-		(lib_id "power:VCC")
-		(at 87.63 118.745 0)
-		(unit 1)
-		(exclude_from_sim no)
-		(in_bom yes)
-		(on_board yes)
-		(dnp no)
-		(fields_autoplaced yes)
-		(property "Reference" "#PWR028"
-			(at 87.63 122.555 0)
-			(effects
-				(font
-					(size 1.27 1.27)
-				)
-				(hide yes)
-			)
-		)
-		(property "Value" "VCC"
-			(at 87.63 113.665 0)
-			(effects
-				(font
-					(size 1.27 1.27)
-				)
-			)
-		)
-		(property "Footprint" ""
-			(at 87.63 118.745 0)
-			(effects
-				(font
-					(size 1.27 1.27)
-				)
-				(hide yes)
-			)
-		)
-		(property "Datasheet" ""
-			(at 87.63 118.745 0)
-			(effects
-				(font
-					(size 1.27 1.27)
-				)
-				(hide yes)
-			)
-		)
-		(property "Description" "Power symbol creates a global label with name \"VCC\""
-			(at 87.63 118.745 0)
-			(effects
-				(font
-					(size 1.27 1.27)
-				)
-				(hide yes)
-			)
-		)
-		(pin "1"
-		)
-		(instances
-			(project "ECE 411 Project"
-				(path "/2625e5a1-d0c8-41ce-941d-75d035a5f1c5/fc48e9dd-306b-4a9b-831b-312573108cdc"
-					(reference "#PWR028")
-					(unit 1)
-				)

Commit message: schematic update
Parts:
- C33: value .1uF -> 0.1uF
Changed lines of the file:
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@@
 			)
 		)
-		(property "Value" ".1uF"
+		(property "Value" "0.1uF"
 			(at 129.54 114.9349 0)
 			(effects

Commit message: pcb amp revision
Parts:
- L1, L2: footprint Inductor-VLS6045AF_330M:IND_VLS6045AF-330M -> Inductor_THT:RL110-330K-RC
Changed lines of the file:
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@@
 			)
 		)
-		(property "Footprint" "Inductor-VLS6045AF_330M:IND_VLS6045AF-330M"
+		(property "Footprint" "Inductor_THT:RL110-330K-RC"
 			(at 193.04 105.41 0)
 			(effects
@@
 		(on_board yes)
 		(dnp no)
-		(fields_autoplaced yes)
 		(property "Reference" "C32"
-			(at 127.635 77.47 0)
+			(at 116.84 77.47 0)
 			(effects
 				(font
@@
 		)
 		(property "Value" "1uF"
-			(at 127.635 80.01 0)
+			(at 116.84 80.01 0)
 			(effects
 				(font
@@
 			)
 		)
-		(property "Footprint" "Inductor-VLS6045AF_330M:IND_VLS6045AF-330M"
+		(property "Footprint" "Inductor_THT:RL110-330K-RC"
 			(at 193.04 86.36 0)
 			(effects

Commit message: add testpoints
Parts:
- GND1, SPK+1, SPK-1: footprint TestPoint:TestPoint_Bridge_Pitch2.0mm_Drill0.7mm -> TestPoint:TestPoint_Loop_D3.80mm_Drill2.5mm
Changed lines of the file:
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@@
 			)
 		)
-		(property "Footprint" "TestPoint:TestPoint_Bridge_Pitch2.0mm_Drill0.7mm"
+		(property "Footprint" "TestPoint:TestPoint_Loop_D3.80mm_Drill2.5mm"
 			(at 24.13 24.765 0)
 			(effects
@@
 			)
 		)
-		(property "Footprint" "TestPoint:TestPoint_Bridge_Pitch2.0mm_Drill0.7mm"
+		(property "Footprint" "TestPoint:TestPoint_Loop_D3.80mm_Drill2.5mm"
 			(at 202.565 105.41 0)
 			(effects
@@
 			)
 		)
-		(property "Footprint" "TestPoint:TestPoint_Bridge_Pitch2.0mm_Drill0.7mm"
+		(property "Footprint" "TestPoint:TestPoint_Loop_D3.80mm_Drill2.5mm"
 			(at 202.565 86.36 0)
 			(effects
