File: Electrical Design/Modules/ECE 411 Project/Amp.kicad_sch (KiCad schematic)
At the start: 22 parts, among them U9 TPA3136D2PWPR

Commit message: minor formatting updates
Parts:
- C24, C25, C26, C27, C28, C29, C30, C31, C32, C33, C36, C37, GND1, R40, R43, SPK+1, SPK-1: Part Origin DK -> (none); Part_Origin (none) -> DK
- C34, C35: On Hand (On Way) (100) -> (none); On_Hand_(On_Way) (none) -> (100); Part Number 1276-1074-1-ND -> (none); Part Origin DK -> (none); Part_Number (none) -> 1276-1074-1-ND; Part_Origin (none) -> DK
- U9: Part Origin SBP -> (none); Part_Origin (none) -> SBP
