File: Electrical Design/Modules/ECE 411 Project/Tremolo.kicad_sch (KiCad schematic)
At the start: 7 parts, among them U4 NE555D, U5 LTV-827

Commit message: pcb amp revision
Parts:
- RV6: footprint Connector_PinSocket_2.54mm:PinSocket_1x03_P2.54mm_Vertical -> Connector_PinSocket_2.54mm:PinSocket_1x02_P2.54mm_Vertical
Changed lines of the file:
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@@
 			)
 		)
-		(property "Footprint" "Connector_PinSocket_2.54mm:PinSocket_1x03_P2.54mm_Vertical"
+		(property "Footprint" "Connector_PinSocket_2.54mm:PinSocket_1x02_P2.54mm_Vertical"
 			(at 149.86 89.535 0)
 			(effects

Commit message: minor formatting updates
Parts:
- C2: On Hand (On Way) (100) -> (none); On_Hand_(On_Way) (none) -> (100); Part Number CL31B475KAHNNNE -> (none); Part Origin DK -> (none); Part_Number (none) -> CL31B475KAHNNNE; Part_Origin (none) -> DK
- D3, R1, R2, RV6, U4: Part Origin DK -> (none); Part_Origin (none) -> DK
- U5: Part Origin SBP -> (none); Part_Origin (none) -> SBP
Changed lines of the file:
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@@
 			)
 		)
-		(property "Part Number" ""
-			(at 135.255 116.205 0)
-			(effects
-				(font
-					(size 1.27 1.27)
-				)
-				(hide yes)
-			)
-		)
-		(property "Part Origin" "DK"
-			(at 135.255 116.205 0)
-			(effects
-				(font
-					(size 1.27 1.27)
-				)
-				(hide yes)
-			)
-		)
-		(property "On Hand (On Way)" ""
+		(property "Part_Origin" "DK"
 			(at 135.255 116.205 0)
 			(effects
@@
 			)
 		)
-		(property "Part Number" "CL31B475KAHNNNE"
+		(property "On_Hand_(On_Way)" "(100)"
 			(at 112.395 103.505 0)
 			(effects
@@
 			)
 		)
-		(property "Part Origin" "DK"
+		(property "Part_Number" "CL31B475KAHNNNE"
 			(at 112.395 103.505 0)
 			(effects
@@
 			)
 		)
-		(property "On Hand (On Way)" "(100)"
+		(property "Part_Origin" "DK"
 			(at 112.395 103.505 0)
 			(effects
@@
 			)
 		)
-		(property "Part Number" ""
-			(at 140.335 94.615 0)
-			(effects
-				(font
-					(size 1.27 1.27)
-				)
-				(hide yes)
-			)
-		)
-		(property "Part Origin" "DK"
-			(at 140.335 94.615 0)
-			(effects
-				(font
-					(size 1.27 1.27)
-				)
-				(hide yes)
-			)
-		)
-		(property "On Hand (On Way)" ""
+		(property "Part_Origin" "DK"
 			(at 140.335 94.615 0)
 			(effects
@@
 			)
 		)
-		(property "Part Number" ""
-			(at 149.86 89.535 0)
-			(effects
-				(font
-					(size 1.27 1.27)
-				)
-				(hide yes)
-			)
-		)
-		(property "Part Origin" "DK"
-			(at 149.86 89.535 0)
-			(effects
-				(font
-					(size 1.27 1.27)
-				)
-				(hide yes)
-			)
-		)
-		(property "On Hand (On Way)" ""
+		(property "Part_Origin" "DK"
 			(at 149.86 89.535 0)
 			(effects
@@
 			)
 		)
-		(property "Part Number" ""
-			(at 166.37 111.125 0)
-			(effects
-				(font
-					(size 1.27 1.27)
-				)
-				(hide yes)
-			)
-		)
-		(property "Part Origin" "DK"
-			(at 166.37 111.125 0)
-			(effects
-				(font
-					(size 1.27 1.27)
-				)
-				(hide yes)
-			)
-		)
-		(property "On Hand (On Way)" ""
+		(property "Part_Origin" "DK"
 			(at 166.37 111.125 0)
 			(effects
@@
 			)
 		)
-		(property "Part Number" ""
-			(at 158.75 124.46 0)
-			(effects
-				(font
-					(size 1.27 1.27)
-				)
-				(hide yes)
-			)
-		)
-		(property "Part Origin" "DK"
-			(at 158.75 124.46 0)
-			(effects
-				(font
-					(size 1.27 1.27)
-				)
-				(hide yes)
-			)
-		)
-		(property "On Hand (On Way)" ""
+		(property "Part_Origin" "DK"
 			(at 158.75 124.46 0)
 			(effects
@@
 			)
 		)
-		(property "Part Number" ""
+		(property "Part_Origin" "SBP"
 			(at 180.34 113.665 0)
 			(effects
-				(font
-					(size 1.27 1.27)
-				)
-				(hide yes)
-			)
-		)
-		(property "Part Origin" "SBP"
-			(at 180.34 113.665 0)
-			(effects
-				(font
-					(size 1.27 1.27)
-				)
-				(hide yes)
-			)
-		)
-		(property "On Hand (On Way)" ""
-			(at 180.34 113.665 0)
-			(effects
